File: split_keeb/split_keeb.kicad_sch (KiCad schematic)
At the start: 0 parts

Commit message: add libraries
Other:
- added sheet Right (side.kicad_sch)
- added sheet left (half.kicad_sch)
Changed lines of the file:
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@@
 	(generator_version "9.0")
 	(paper "A4")
+	(sheet
+		(at 27.94 41.91)
+		(size 99.06 78.74)
+		(exclude_from_sim no)
+		(in_bom yes)
+		(on_board yes)
+		(dnp no)
+		(fields_autoplaced yes)
+		(stroke
+			(width 0.1524)
+			(type solid)
+		)
+		(fill
+			(color 0 0 0 0.0000)
+		)
+		(property "Sheetname" "left"
+			(at 27.94 41.1984 0)
+			(effects
+				(font
+					(size 1.27 1.27)
+				)
+				(justify left bottom)
+			)
+		)
+		(property "Sheetfile" "half.kicad_sch"
+			(at 27.94 121.2346 0)
+			(effects
+				(font
+					(size 1.27 1.27)
+				)
+				(justify left top)
+			)
+		)
+		(instances
+			(project "split_keeb"
+				(path "/2629a1a5-f1c0-4d6e-825a-cf5cf79bde40"
+					(page "2")
+				)
+			)
+		)
+	)
+	(sheet
+		(at 149.86 43.18)
+		(size 116.84 73.66)
+		(exclude_from_sim no)
+		(in_bom yes)
+		(on_board yes)
+		(dnp no)
+		(fields_autoplaced yes)
+		(stroke
+			(width 0.1524)
+			(type solid)
+		)
+		(fill
+			(color 0 0 0 0.0000)
+		)
+		(property "Sheetname" "Right"
+			(at 149.86 42.4684 0)
+			(effects
+				(font
+					(size 1.27 1.27)
+				)
+				(justify left bottom)
+			)
+		)
+		(property "Sheetfile" "side.kicad_sch"
+			(at 149.86 117.4246 0)
+			(effects
+				(font
+					(size 1.27 1.27)
+				)
+				(justify left top)
+			)
+		)
+		(instances
+			(project "split_keeb"
+				(path "/2629a1a5-f1c0-4d6e-825a-cf5cf79bde40"
+					(page "3")
+				)
+			)
+		)
+	)
 	(sheet_instances
 		(path "/"
